File: PCB/arducard.brd (EAGLE design)
At the start: 82.3 x 45.8 mm, 90 parts, among them J1 USB MICRO, J3 051296-4094, Q1 BSS84, Q10 DMG2301U-7, Q2 BC817-16LT1SMD, Q3 DMG2301U-7, Q4 2N7002, Q5 BSS84, Q6 2N7002, Q7 2N7002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

Commit message: renamed a part
Parts:
- J1: value USB MICRO -> USB MICRO B
Changed lines of the file:
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@@
 <element name="Z2" library="varistor" package="CT/CN0603" value="CG0603MLC-05E" x="74.561" y="10.56" rot="R180"/>
 <element name="C9" library="SmartPrj" package="C0603-ROUND" value="100n" x="69.35" y="7.773" rot="R90"/>
-<element name="J1" library="SmartPrj" package="CON2_USB_MICRO_B_AT" value="USB MICRO" x="80.733" y="14.143" smashed="yes" rot="R90"/>
+<element name="J1" library="SmartPrj" package="CON2_USB_MICRO_B_AT" value="USB MICRO B" x="80.733" y="14.143" smashed="yes" rot="R90"/>
 <element name="U1" library="SmartPrj" package="TQFP44-PAD" value="ATMEGA32U4-XUAU" x="59.68" y="14.103" rot="R180"/>
 <element name="C14" library="SmartPrj" package="C0603-ROUND" value="1uF" x="73.955" y="40.622"/>
